Commit message: lowered IMU link to 0.056 m from 0.069 m

File: src/amr_description/urdf/amr.urdf.xacro (robot description, xacro)
@@ -209,5 +209,5 @@
     </link>
     <joint name="imu_joint" type="fixed">
-        <origin xyz="0 0 0.0698986241758014" rpy="0 0 0" />
+        <origin xyz="0 0 0.053" rpy="0 0 0" />
         <parent link="base_link" />
         <child link="imu_link" />
